Commit message: wys work

File: src/tergeo_description/urdf/macro/cfg/cfg_lidar.xacro (robot description, xacro)
@@ -6,5 +6,5 @@
   <xacro:property name="PI" value="3.1415926535897931" />
   <!-- Lidar intrinsic -->
-  <xacro:property name="h_sample" value="90" />
+  <xacro:property name="h_sample" value="2100" />
   <xacro:property name="h_min_angle" value="${-180 *PI/180.0}" />
   <xacro:property name="h_max_angle" value="${+180 *PI/180.0}" />

File: src/tergeo_description/urdf/macro/model_lidar.xacro (robot description, xacro)
@@ -44,5 +44,5 @@
             <horizontal>
               <samples>${lidar.h_sample}</samples>
-              <resolution>6</resolution>
+              <resolution>1</resolution>
               <min_angle>${lidar.h_min_angle}</min_angle>
               <max_angle>${lidar.h_max_angle}</max_angle>
@@ -68,5 +68,5 @@
         <plugin name="lidar_sensor" filename="libgazebo_ros_velodyne_laser.so">
           <topicName>${lidar.pub_topic_name}</topicName>
-          <frameName>${lidar_name}_link</frameName>
+          <frameName>top_lidar16_link</frameName>
           <min_range>${lidar.min_range}</min_range>
           <max_range>${lidar.max_range}</max_range>
